Commit message: revised walk training for landau model

File: algorithms/urdf_learn_wasd_walk/inputs/landau_v10/landau_v10_parallel_mesh.urdf (robot description, URDF)
Before this commit: robot landau_v10_parallel_mesh, 69 links, 68 joints
Links:
- link foot_l: geometry collision box size=0.056000 0.088000 0.018000; visual mesh filename=mesh_collision_stl/landau_v10/foot_l.stl
- link foot_r: geometry collision box size=0.056000 0.088000 0.018000; visual mesh filename=mesh_collision_stl/landau_v10/foot_r.stl
- link toes_01_l: geometry collision box size=0.044000 0.038000 0.012000; visual mesh filename=mesh_collision_stl/landau_v10/toes_01_l.stl
- link toes_01_r: geometry collision box size=0.044000 0.038000 0.012000; visual mesh filename=mesh_collision_stl/landau_v10/toes_01_r.stl
