Commit message: continue traning urdf walking

File: algorithms/urdf_learn_wasd_walk/inputs/landau_v10/landau_v10_parallel_mesh.urdf (robot description, URDF)
Before this commit: robot landau_v10_parallel_mesh, 69 links, 68 joints
Links:
- added link left_hip_roll_link, mass 0.020000
- added link right_hip_roll_link, mass 0.020000
- link arm_stretch_l: geometry 
- link arm_stretch_r: geometry 
- link arm_twist_l: mass 0.020000 -> 0.030000; geometry collision mesh filename=mesh_collision_stl/landau_v10/arm_stretch_l.stl; collision mesh filename=mesh_collision_stl/landau_v10/arm_twist_l.stl
- link arm_twist_r: mass 0.020000 -> 0.030000; geometry collision mesh filename=mesh_collision_stl/landau_v10/arm_stretch_r.stl; collision mesh filename=mesh_collision_stl/landau_v10/arm_twist_r.stl
- link foot_l: geometry collision mesh filename=mesh_collision_stl/landau_v10/foot_l.stl; visual mesh filename=mesh_collision_stl/landau_v10/foot_l.stl
- link foot_r: geometry collision mesh filename=mesh_collision_stl/landau_v10/foot_r.stl; visual mesh filename=mesh_collision_stl/landau_v10/foot_r.stl
- link forearm_stretch_l: mass 0.030000 -> 0.050000; geometry collision mesh filename=mesh_collision_stl/landau_v10/forearm_stretch_l.stl; collision mesh filename=mesh_collision_stl/landau_v10/forearm_twist_l.stl
- link forearm_stretch_r: mass 0.030000 -> 0.050000; geometry collision mesh filename=mesh_collision_stl/landau_v10/forearm_stretch_r.stl; collision mesh filename=mesh_collision_stl/landau_v10/forearm_twist_r.stl
- link forearm_twist_l: geometry 
- link forearm_twist_r: geometry 
- link leg_stretch_l: mass 0.057288 -> 0.020000; geometry 
- link leg_stretch_r: mass 0.057287 -> 0.020000; geometry 
- link leg_twist_l: mass 0.020000 -> 0.077288; geometry collision mesh filename=mesh_collision_stl/landau_v10/leg_stretch_l.stl; collision mesh filename=mesh_collision_stl/landau_v10/leg_twist_l.stl
- link leg_twist_r: mass 0.020000 -> 0.077287; geometry collision mesh filename=mesh_collision_stl/landau_v10/leg_stretch_r.stl; collision mesh filename=mesh_collision_stl/landau_v10/leg_twist_r.stl
- link spine_01_x: geometry 
- link spine_02_x: geometry 
- link spine_03_x: mass 0.040000 -> 0.080000; geometry collision mesh filename=mesh_collision_stl/landau_v10/spine_01_x.stl; collision mesh filename=mesh_collision_stl/landau_v10/spine_02_x.stl
- link thigh_stretch_l: mass 0.041351 -> 0.020000; geometry 
- link thigh_stretch_r: mass 0.041351 -> 0.020000; geometry 
- link thigh_twist_l: mass 0.020000 -> 0.051351; geometry collision mesh filename=mesh_collision_stl/landau_v10/thigh_stretch_l.stl; collision mesh filename=mesh_collision_stl/landau_v10/thigh_twist_l.stl
- link thigh_twist_r: mass 0.020000 -> 0.051351; geometry collision mesh filename=mesh_collision_stl/landau_v10/thigh_stretch_r.stl; collision mesh filename=mesh_collision_stl/landau_v10/thigh_twist_r.stl
- link toes_01_l: geometry collision mesh filename=mesh_collision_stl/landau_v10/toes_01_l.stl; visual mesh filename=mesh_collision_stl/landau_v10/toes_01_l.stl
- link toes_01_r: geometry collision mesh filename=mesh_collision_stl/landau_v10/toes_01_r.stl; visual mesh filename=mesh_collision_stl/landau_v10/toes_01_r.stl
Joints:
- removed joint arm_stretch_l
- removed joint arm_stretch_r
- removed joint arm_twist_l
- removed joint arm_twist_r
- removed joint foot_l
- removed joint foot_r
- removed joint forearm_stretch_l
- removed joint forearm_stretch_r
- removed joint forearm_twist_l
- removed joint forearm_twist_r
- removed joint hand_l
- removed joint hand_r
- removed joint head_x
- removed joint index1_base_l
- removed joint index1_base_r
- removed joint index1_l
- removed joint index1_r
- removed joint index2_l
- removed joint index2_r
- removed joint index3_l
- removed joint index3_r
- removed joint leg_stretch_l
- removed joint leg_stretch_r
- removed joint leg_twist_l
- removed joint leg_twist_r
- removed joint middle1_base_l
- removed joint middle1_base_r
- removed joint middle1_l
- removed joint middle1_r
- removed joint middle2_l
- removed joint middle2_r
- removed joint middle3_l
- removed joint middle3_r
- removed joint neck_x
- removed joint pinky1_base_l
- removed joint pinky1_base_r
- removed joint pinky1_l
- removed joint pinky1_r
- removed joint pinky2_l
- removed joint pinky2_r
- removed joint pinky3_l
- removed joint pinky3_r
- removed joint ring1_base_l
- removed joint ring1_base_r
- removed joint ring1_l
- removed joint ring1_r
- removed joint ring2_l
- removed joint ring2_r
- removed joint ring3_l
- removed joint ring3_r
- removed joint shoulder_l
- removed joint shoulder_r
- removed joint spine_01_x
- removed joint spine_02_x
- removed joint spine_03_x
- removed joint thigh_stretch_l
- removed joint thigh_stretch_r
- removed joint thigh_twist_l
- removed joint thigh_twist_r
- removed joint thumb1_l
- removed joint thumb1_r
- removed joint thumb2_l
- removed joint thumb2_r
- removed joint thumb3_l
- removed joint thumb3_r
- removed joint toes_01_l
- removed joint toes_01_r
- added joint head_yaw_joint: type revolute, parent neck_x, child head_x, origin xyz=0.000000 0.039366 0.000000 rpy=-0.221063 0.000000 0.000000, axis -0.000000 0.991039 -0.133576, limit lower=-0.700000 upper=0.700000 effort=50.0 velocity=4.0
- added joint left_ankle_pitch_joint: type revolute, parent leg_twist_l, child foot_l, origin xyz=0.000000 0.064923 0.000000 rpy=-3.024146 1.553144 1.878009, axis -0.960401 0.263140 0.091586, limit lower=-0.600000 upper=0.800000 effort=50.0 velocity=4.0
- added joint left_elbow_joint: type revolute, parent arm_twist_l, child forearm_stretch_l, origin xyz=-0.000000 0.090539 0.000000 rpy=0.000064 -0.000235 -0.264238, axis -1.000000 0.000000 0.000000, limit lower=-1.800000 upper=1.800000 effort=50.0 velocity=4.0
- added joint left_forearm_roll_joint: type revolute, parent forearm_stretch_l, child forearm_twist_l, origin xyz=0.000000 0.046099 0.000000 rpy=-0.000000 -0.161408 0.000000, axis 0.000000 1.000000 0.000000, limit lower=-1.200000 upper=1.200000 effort=50.0 velocity=4.0
- added joint left_hip_pitch_joint: type revolute, parent root_x, child thigh_stretch_l, origin xyz=0.059407 0.000000 -0.000000 rpy=2.748947 -1.256079 0.394193, axis 0.285805 0.018900 0.958101, limit lower=-1.800000 upper=1.800000 effort=50.0 velocity=4.0
- added joint left_hip_roll_joint: type revolute, parent thigh_stretch_l, child left_hip_roll_link, origin xyz=-0.000000 -0.000000 0.000000 rpy=-0.000000 0.000000 0.000000, axis -0.958244 0.015230 0.285547, limit lower=-0.700000 upper=0.700000 effort=50.0 velocity=4.0
- added joint left_hip_yaw_joint: type revolute, parent left_hip_roll_link, child thigh_twist_l, origin xyz=-0.000000 0.000000 0.000000 rpy=0.000000 -0.000000 -0.000000, axis -0.009195 -0.999705 0.022463, limit lower=-1.200000 upper=1.200000 effort=50.0 velocity=4.0
- added joint left_index_base_joint: type revolute, parent hand_l, child index1_base_l, origin xyz=0.013064 0.021871 -0.000770 rpy=0.046371 0.000000 -0.093843, axis 1.000000 0.000000 0.000000, limit lower=-0.450000 upper=0.450000 effort=50.0 velocity=4.0
- added joint left_index_distal_joint: type revolute, parent index2_l, child index3_l, origin xyz=0.000000 0.014291 0.000000 rpy=0.043239 0.002466 -0.001454, axis 0.985696 0.168073 -0.012468, limit lower=-1.600000 upper=0.000000 effort=50.0 velocity=4.0
- added joint left_index_intermediate_joint: type revolute, parent index1_l, child index2_l, origin xyz=0.000000 0.014229 0.000000 rpy=0.015110 0.000839 0.132563, axis 0.985924 0.167021 -0.007622, limit lower=-1.600000 upper=0.000000 effort=50.0 velocity=4.0
- added joint left_index_proximal_joint: type revolute, parent index1_base_l, child index1_l, origin xyz=0.000000 0.041832 -0.000000 rpy=-0.018912 0.000823 -0.094255, axis 0.955180 0.295965 -0.005925, limit lower=-1.600000 upper=0.000000 effort=50.0 velocity=4.0
- added joint left_knee_joint: type revolute, parent thigh_twist_l, child leg_stretch_l, origin xyz=0.000000 0.129607 -0.000000 rpy=-0.000000 -0.000000 0.264397, axis 0.280812 -0.056446 0.958101, limit lower=-1.800000 upper=1.800000 effort=50.0 velocity=4.0
- added joint left_middle_base_joint: type revolute, parent hand_l, child middle1_base_l, origin xyz=0.001299 0.023015 -0.000209 rpy=0.004885 -0.000000 0.030411, axis 1.000000 0.000000 0.000000, limit lower=-0.450000 upper=0.450000 effort=50.0 velocity=4.0
- added joint left_middle_distal_joint: type revolute, parent middle2_l, child middle3_l, origin xyz=-0.000000 0.012887 -0.000000 rpy=-0.050883 0.004692 -0.002267, axis 0.999693 0.019565 0.015181, limit lower=-1.600000 upper=0.000000 effort=50.0 velocity=4.0
- added joint left_middle_intermediate_joint: type revolute, parent middle1_l, child middle2_l, origin xyz=0.000000 0.017378 -0.000000 rpy=-0.079008 0.007453 0.057353, axis 0.999792 0.018045 0.009475, limit lower=-1.600000 upper=0.000000 effort=50.0 velocity=4.0
- added joint left_middle_proximal_joint: type revolute, parent middle1_base_l, child middle1_l, origin xyz=0.000000 0.042722 -0.000000 rpy=-0.034946 0.001127 0.006071, axis 0.997106 0.076017 0.000570, limit lower=-1.600000 upper=0.000000 effort=50.0 velocity=4.0
- added joint left_pinky_base_joint: type revolute, parent hand_l, child pinky1_base_l, origin xyz=-0.016800 0.017932 -0.000631 rpy=-0.137206 -0.000000 0.242037, axis 1.000000 0.000000 0.000000, limit lower=-0.450000 upper=0.450000 effort=50.0 velocity=4.0
- added joint left_pinky_distal_joint: type revolute, parent pinky2_l, child pinky3_l, origin xyz=0.000000 0.007725 0.000000 rpy=-0.035199 0.021262 -0.013497, axis 0.901025 -0.430231 0.055273, limit lower=-1.600000 upper=0.000000 effort=50.0 velocity=4.0
- added joint left_pinky_intermediate_joint: type revolute, parent pinky1_l, child pinky2_l, origin xyz=-0.000000 0.007820 0.000000 rpy=-0.117001 0.072529 -0.016065, axis 0.896459 -0.440159 0.051207, limit lower=-1.600000 upper=0.000000 effort=50.0 velocity=4.0
- added joint left_pinky_proximal_joint: type revolute, parent pinky1_base_l, child pinky1_l, origin xyz=-0.000000 0.043247 -0.000000 rpy=-0.175045 0.149489 0.319301, axis 0.894467 -0.445599 0.037007, limit lower=-1.600000 upper=0.000000 effort=50.0 velocity=4.0
- added joint left_ring_base_joint: type revolute, parent hand_l, child ring1_base_l, origin xyz=-0.008684 0.021505 -0.000181 rpy=-0.052344 -0.000000 0.122979, axis 1.000000 0.000000 0.000000, limit lower=-0.450000 upper=0.450000 effort=50.0 velocity=4.0
- added joint left_ring_distal_joint: type revolute, parent ring2_l, child ring3_l, origin xyz=0.000000 0.011927 0.000000 rpy=0.019436 -0.006208 -0.021339, axis 0.980156 -0.197141 0.020733, limit lower=-1.600000 upper=0.000000 effort=50.0 velocity=4.0
- added joint left_ring_intermediate_joint: type revolute, parent ring1_l, child ring2_l, origin xyz=-0.000000 0.013621 -0.000000 rpy=-0.131789 0.045045 0.064214, axis 0.975595 -0.218373 0.022982, limit lower=-1.600000 upper=0.000000 effort=50.0 velocity=4.0
- added joint left_ring_proximal_joint: type revolute, parent ring1_base_l, child ring1_l, origin xyz=-0.000000 0.043050 -0.000000 rpy=-0.036781 0.016557 0.140266, axis 0.988607 -0.150330 0.007495, limit lower=-1.600000 upper=0.000000 effort=50.0 velocity=4.0
- added joint left_shin_roll_joint: type revolute, parent leg_stretch_l, child leg_twist_l, origin xyz=-0.000000 0.064923 0.000000 rpy=-0.000000 0.000000 -0.000000, axis 0.000000 1.000000 0.000000, limit lower=-1.200000 upper=1.200000 effort=50.0 velocity=4.0
- added joint left_shoulder_lift_joint: type revolute, parent spine_03_x, child shoulder_l, origin xyz=0.015987 0.029273 -0.002075 rpy=-0.000093 -1.565935 -1.570703, axis -0.991294 0.000000 -0.131667, limit lower=-1.800000 upper=1.800000 effort=50.0 velocity=4.0
- added joint left_shoulder_pitch_joint: type revolute, parent shoulder_l, child arm_stretch_l, origin xyz=-0.000000 0.047960 -0.000000 rpy=-0.903354 0.052291 0.039342, axis 0.039278 0.616885 0.786072, limit lower=-1.800000 upper=1.800000 effort=50.0 velocity=4.0
- added joint left_thumb_distal_joint: type revolute, parent thumb2_l, child thumb3_l, origin xyz=-0.000000 0.016161 -0.000000 rpy=0.068861 0.078468 0.099511, axis -0.130429 0.598210 0.790654, limit lower=-1.500000 upper=1.000000 effort=50.0 velocity=4.0
- added joint left_thumb_metacarpal_joint: type revolute, parent hand_l, child thumb1_l, origin xyz=0.014072 0.021172 -0.009160 rpy=-1.356045 1.216473 -1.928883, axis 0.980893 -0.000001 0.194550, limit lower=-1.200000 upper=1.200000 effort=50.0 velocity=4.0
- added joint left_thumb_proximal_joint: type revolute, parent thumb1_l, child thumb2_l, origin xyz=0.000000 0.027022 -0.000000 rpy=0.069783 -0.348140 -0.462812, axis -0.118534 0.533252 0.837611, limit lower=-1.500000 upper=1.000000 effort=50.0 velocity=4.0
- added joint left_toe_joint: type revolute, parent foot_l, child toes_01_l, origin xyz=-0.000000 0.064823 0.000000 rpy=-2.796910 0.000186 -3.141524, axis 0.960365 0.216718 -0.175304, limit lower=-0.600000 upper=0.800000 effort=50.0 velocity=4.0
- added joint left_upper_arm_roll_joint: type revolute, parent arm_stretch_l, child arm_twist_l, origin xyz=0.000000 0.000000 -0.000000 rpy=0.000000 -0.000000 -0.000000, axis 0.000000 1.000000 0.000000, limit lower=-1.200000 upper=1.200000 effort=50.0 velocity=4.0
- added joint left_wrist_pitch_joint: type revolute, parent forearm_twist_l, child hand_l, origin xyz=-0.000000 0.046099 0.000000 rpy=-0.012699 -0.000001 0.120527, axis 0.077713 0.590646 0.803180, limit lower=-1.800000 upper=1.800000 effort=50.0 velocity=4.0
- added joint neck_pitch_joint: type revolute, parent spine_03_x, child neck_x, origin xyz=-0.000000 0.069467 0.000000 rpy=0.227851 0.000000 -0.000000, axis 1.000000 0.000000 -0.000000, limit lower=-0.700000 upper=0.700000 effort=50.0 velocity=4.0
- added joint right_ankle_pitch_joint: type revolute, parent leg_twist_r, child foot_r, origin xyz=0.000000 0.064923 -0.000000 rpy=-3.024103 -1.553146 -1.878052, axis -0.960401 -0.263139 -0.091588, limit lower=-0.600000 upper=0.800000 effort=50.0 velocity=4.0
- added joint right_elbow_joint: type revolute, parent arm_twist_r, child forearm_stretch_r, origin xyz=0.000000 0.090539 0.000000 rpy=-0.000047 -0.000173 0.264238, axis 1.000000 0.000000 0.000000, limit lower=-1.800000 upper=1.800000 effort=50.0 velocity=4.0
- added joint right_forearm_roll_joint: type revolute, parent forearm_stretch_r, child forearm_twist_r, origin xyz=-0.000000 0.046099 0.000000 rpy=-0.000000 0.161409 -0.000000, axis 0.000000 1.000000 0.000000, limit lower=-1.200000 upper=1.200000 effort=50.0 velocity=4.0
- added joint right_hip_pitch_joint: type revolute, parent root_x, child thigh_stretch_r, origin xyz=-0.059407 0.000000 0.000000 rpy=2.748940 1.256084 -0.394200, axis 0.285805 -0.018900 -0.958101, limit lower=-1.800000 upper=1.800000 effort=50.0 velocity=4.0
- added joint right_hip_roll_joint: type revolute, parent thigh_stretch_r, child right_hip_roll_link, origin xyz=-0.000000 -0.000000 -0.000000 rpy=0.000000 -0.000000 0.000000, axis 0.958244 0.015230 0.285547, limit lower=-0.700000 upper=0.700000 effort=50.0 velocity=4.0
- added joint right_hip_yaw_joint: type revolute, parent right_hip_roll_link, child thigh_twist_r, origin xyz=0.000000 0.000000 0.000000 rpy=0.000000 0.000000 -0.000000, axis 0.009195 -0.999705 0.022463, limit lower=-1.200000 upper=1.200000 effort=50.0 velocity=4.0
- added joint right_index_base_joint: type revolute, parent hand_r, child index1_base_r, origin xyz=-0.013064 0.021871 -0.000770 rpy=0.046371 -0.000000 0.093843, axis 1.000000 0.000000 0.000000, limit lower=-0.450000 upper=0.450000 effort=50.0 velocity=4.0
- added joint right_index_distal_joint: type revolute, parent index2_r, child index3_r, origin xyz=0.000000 0.014291 0.000000 rpy=0.043239 -0.002465 0.001454, axis 0.985696 -0.168074 0.012467, limit lower=-1.600000 upper=0.000000 effort=50.0 velocity=4.0
- added joint right_index_intermediate_joint: type revolute, parent index1_r, child index2_r, origin xyz=0.000000 0.014229 0.000000 rpy=0.015109 -0.000840 -0.132563, axis 0.985924 -0.167022 0.007621, limit lower=-1.600000 upper=0.000000 effort=50.0 velocity=4.0
- added joint right_index_proximal_joint: type revolute, parent index1_base_r, child index1_r, origin xyz=0.000000 0.041832 -0.000000 rpy=-0.018911 -0.000823 0.094256, axis 0.955180 -0.295966 0.005924, limit lower=-1.600000 upper=0.000000 effort=50.0 velocity=4.0
- added joint right_knee_joint: type revolute, parent thigh_twist_r, child leg_stretch_r, origin xyz=0.000000 0.129607 0.000000 rpy=-0.000000 0.000000 -0.264397, axis 0.280812 0.056446 -0.958101, limit lower=-1.800000 upper=1.800000 effort=50.0 velocity=4.0
- added joint right_middle_base_joint: type revolute, parent hand_r, child middle1_base_r, origin xyz=-0.001299 0.023015 -0.000209 rpy=0.004885 0.000000 -0.030411, axis 1.000000 0.000000 0.000000, limit lower=-0.450000 upper=0.450000 effort=50.0 velocity=4.0
- added joint right_middle_distal_joint: type revolute, parent middle2_r, child middle3_r, origin xyz=-0.000000 0.012887 -0.000000 rpy=-0.050882 -0.004692 0.002267, axis 0.999693 -0.019566 -0.015182, limit lower=-1.600000 upper=0.000000 effort=50.0 velocity=4.0
- added joint right_middle_intermediate_joint: type revolute, parent middle1_r, child middle2_r, origin xyz=-0.000000 0.017378 -0.000000 rpy=-0.079009 -0.007453 -0.057353, axis 0.999792 -0.018046 -0.009476, limit lower=-1.600000 upper=0.000000 effort=50.0 velocity=4.0
- added joint right_middle_proximal_joint: type revolute, parent middle1_base_r, child middle1_r, origin xyz=0.000000 0.042722 -0.000000 rpy=-0.034946 -0.001128 -0.006071, axis 0.997106 -0.076018 -0.000571, limit lower=-1.600000 upper=0.000000 effort=50.0 velocity=4.0
- added joint right_pinky_base_joint: type revolute, parent hand_r, child pinky1_base_r, origin xyz=0.016800 0.017932 -0.000631 rpy=-0.137207 -0.000000 -0.242037, axis 1.000000 0.000000 0.000000, limit lower=-0.450000 upper=0.450000 effort=50.0 velocity=4.0
- added joint right_pinky_distal_joint: type revolute, parent pinky2_r, child pinky3_r, origin xyz=-0.000000 0.007725 -0.000000 rpy=-0.035197 -0.021263 0.013498, axis 0.901025 0.430232 -0.055275, limit lower=-1.600000 upper=0.000000 effort=50.0 velocity=4.0
- added joint right_pinky_intermediate_joint: type revolute, parent pinky1_r, child pinky2_r, origin xyz=0.000000 0.007821 -0.000000 rpy=-0.117003 -0.072529 0.016065, axis 0.896458 0.440160 -0.051208, limit lower=-1.600000 upper=0.000000 effort=50.0 velocity=4.0
- added joint right_pinky_proximal_joint: type revolute, parent pinky1_base_r, child pinky1_r, origin xyz=0.000000 0.043247 0.000000 rpy=-0.175045 -0.149489 -0.319301, axis 0.894467 0.445599 -0.037008, limit lower=-1.600000 upper=0.000000 effort=50.0 velocity=4.0
- added joint right_ring_base_joint: type revolute, parent hand_r, child ring1_base_r, origin xyz=0.008684 0.021505 -0.000181 rpy=-0.052344 0.000000 -0.122979, axis 1.000000 0.000000 0.000000, limit lower=-0.450000 upper=0.450000 effort=50.0 velocity=4.0
- added joint right_ring_distal_joint: type revolute, parent ring2_r, child ring3_r, origin xyz=-0.000000 0.011927 0.000000 rpy=0.019436 0.006209 0.021339, axis 0.980156 0.197140 -0.020734, limit lower=-1.600000 upper=0.000000 effort=50.0 velocity=4.0
- added joint right_ring_intermediate_joint: type revolute, parent ring1_r, child ring2_r, origin xyz=-0.000000 0.013621 0.000000 rpy=-0.131790 -0.045046 -0.064214, axis 0.975595 0.218373 -0.022983, limit lower=-1.600000 upper=0.000000 effort=50.0 velocity=4.0
- added joint right_ring_proximal_joint: type revolute, parent ring1_base_r, child ring1_r, origin xyz=0.000000 0.043050 -0.000000 rpy=-0.036781 -0.016557 -0.140266, axis 0.988607 0.150330 -0.007496, limit lower=-1.600000 upper=0.000000 effort=50.0 velocity=4.0
- added joint right_shin_roll_joint: type revolute, parent leg_stretch_r, child leg_twist_r, origin xyz=-0.000000 0.064923 -0.000000 rpy=-0.000000 0.000000 -0.000000, axis 0.000000 1.000000 0.000000, limit lower=-1.200000 upper=1.200000 effort=50.0 velocity=4.0
- added joint right_shoulder_lift_joint: type revolute, parent spine_03_x, child shoulder_r, origin xyz=-0.015987 0.029273 -0.002075 rpy=0.000033 1.565935 1.570829, axis 0.991294 0.000000 -0.131667, limit lower=-1.800000 upper=1.800000 effort=50.0 velocity=4.0
- added joint right_shoulder_pitch_joint: type revolute, parent shoulder_r, child arm_stretch_r, origin xyz=-0.000000 0.047960 0.000000 rpy=-0.903337 -0.052030 -0.039675, axis 0.039611 -0.616886 -0.786055, limit lower=-1.800000 upper=1.800000 effort=50.0 velocity=4.0
- added joint right_thumb_distal_joint: type revolute, parent thumb2_r, child thumb3_r, origin xyz=0.000000 0.016161 -0.000000 rpy=0.068860 -0.078468 -0.099512, axis 0.130429 0.598209 0.790655, limit lower=-1.500000 upper=1.000000 effort=50.0 velocity=4.0
- added joint right_thumb_metacarpal_joint: type revolute, parent hand_r, child thumb1_r, origin xyz=-0.014072 0.021172 -0.009160 rpy=-1.356043 -1.216472 1.928880, axis -0.980893 0.000001 0.194549, limit lower=-1.200000 upper=1.200000 effort=50.0 velocity=4.0
- added joint right_thumb_proximal_joint: type revolute, parent thumb1_r, child thumb2_r, origin xyz=0.000000 0.027022 0.000000 rpy=0.069783 0.348140 0.462812, axis 0.118535 0.533251 0.837611, limit lower=-1.500000 upper=1.000000 effort=50.0 velocity=4.0
- added joint right_toe_joint: type revolute, parent foot_r, child toes_01_r, origin xyz=-0.000000 0.064823 -0.000000 rpy=-2.796910 0.000006 3.141592, axis 0.960401 -0.216718 0.175110, limit lower=-0.600000 upper=0.800000 effort=50.0 velocity=4.0
- added joint right_upper_arm_roll_joint: type revolute, parent arm_stretch_r, child arm_twist_r, origin xyz=0.000000 0.000000 0.000000 rpy=-0.000000 0.000000 0.000000, axis 0.000000 0.000000 1.000000, limit lower=-1.200000 upper=1.200000 effort=50.0 velocity=4.0
- added joint right_wrist_pitch_joint: type revolute, parent forearm_twist_r, child hand_r, origin xyz=0.000000 0.046099 -0.000000 rpy=-0.012698 0.000001 -0.120527, axis 0.077713 -0.590647 -0.803179, limit lower=-1.800000 upper=1.800000 effort=50.0 velocity=4.0
- added joint waist_pitch_joint: type revolute, parent spine_02_x, child spine_03_x, origin xyz=0.000000 0.069307 -0.000000 rpy=-0.284678 -0.000000 0.000000, axis 1.000000 -0.000000 -0.000000, limit lower=-0.700000 upper=0.700000 effort=50.0 velocity=4.0
- added joint waist_roll_joint: type revolute, parent spine_01_x, child spine_02_x, origin xyz=-0.000000 0.067965 -0.000000 rpy=0.352639 0.000000 -0.000000, axis 0.000000 -0.400321 -0.916375, limit lower=-0.700000 upper=0.700000 effort=50.0 velocity=4.0
- added joint waist_yaw_joint: type revolute, parent root_x, child spine_01_x, origin xyz=-0.000000 0.060500 -0.034518 rpy=-0.074748 0.000003 0.000000, axis -0.000000 0.998247 -0.059194, limit lower=-0.700000 upper=0.700000 effort=50.0 velocity=4.0
